File: kicad/treble/treble.kicad_pcb (KiCad board)
At the start: 2 copper layers, 5 parts, among them J1 audio DAC, J2 MICROSD_READER, J3 JOYSTICK, J4 button, U1 ESP32-DevKitC

Commit message: changed a lot in kicad, made all traces on back side
Parts:
- moved J1 61.5 mm to (160.1, 49.1), turned to 0 degrees
- moved J2 32.5 mm to (160.1, 68.7), turned to 0 degrees
- moved J3 19.3 mm to (162.3, 34.9)
- moved J4 13.6 mm to (160.1, 88.2), turned to 0 degrees
- moved U1 8.62 mm to (179.0, 35.5)
Routing:
- net Net-(J3-VRY): track 11.9 -> 78.8 mm, vias 1 -> 0
- net Net-(J3-VRX): track 8.61 -> 68.8 mm, vias 1 -> 0
- net +5V: track 42.8 -> 0.00 mm
- net Net-(J1-LCK): track 52.5 -> 19.3 mm
- net Net-(J4-Pin_1): track 15.4 -> 44.2 mm
- net +3V3: track 64.6 -> 90.4 mm, vias 1 -> 0
- net Net-(J2-MOSI): track 59.6 -> 82.7 mm
- net unconnected-(U1-CHIP_PU-Pad2): track 21.8 -> 0.00 mm
- net Net-(J1-BCK): track 47.8 -> 26.6 mm
- net GND: track 139.2 -> 126.5 mm, vias 1 -> 0
- net Net-(J1-SCK): track 35.5 -> 47.2 mm
- net Net-(J2-MISO): track 42.3 -> 52.7 mm
- net Net-(J2-CLK): track 46.0 -> 52.4 mm
- net Net-(J1-DIN): track 56.1 -> 49.9 mm
- net Net-(J2-CS): track 48.6 -> 53.4 mm, vias 1 -> 0
- added copper zone on B.Cu, net GND
Other:
- board outline added: 55 x 70.5 mm
- board text added: "Anderson"
