File: kicad/treble/treble.kicad_sch (KiCad schematic)
At the start: 5 parts, among them J1 audio DAC, J2 MICROSD_READER, J3 JOYSTICK, J4 button, U1 ESP32-DevKitC

Commit message: changed a lot in kicad, made all traces on back side
Other:
- title: (none) -> Treble
Changed lines of the file:
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@@
 	(generator_version "9.0")
 	(paper "A4")
+	(title_block
+		(title "Treble")
+	)
 	(junction
 		(at 135.89 78.74)
@@
 		)
 		(instances
-			(project ""
+			(project "treble"
 				(path "/3f5034ce-32a3-409e-b32c-964723436806"
 					(reference "U1")
@@
 		)
 		(instances
-			(project ""
+			(project "treble"
 				(path "/3f5034ce-32a3-409e-b32c-964723436806"
 					(reference "#PWR01")
@@
 		)
 		(instances
-			(project ""
+			(project "treble"
 				(path "/3f5034ce-32a3-409e-b32c-964723436806"
 					(reference "#PWR03")
@@
 		)
 		(instances
-			(project ""
+			(project "treble"
 				(path "/3f5034ce-32a3-409e-b32c-964723436806"
 					(reference "J2")
@@
 		)
 		(instances
-			(project ""
+			(project "treble"
 				(path "/3f5034ce-32a3-409e-b32c-964723436806"
 					(reference "#FLG03")
@@
 		)
 		(instances
-			(project ""
+			(project "treble"
 				(path "/3f5034ce-32a3-409e-b32c-964723436806"
 					(reference "#PWR04")
@@
 		)
 		(instances
-			(project ""
+			(project "treble"
 				(path "/3f5034ce-32a3-409e-b32c-964723436806"
 					(reference "#PWR09")
@@
 		)
 		(instances
-			(project ""
+			(project "treble"
 				(path "/3f5034ce-32a3-409e-b32c-964723436806"
 					(reference "#PWR08")
@@
 		)
 		(instances
-			(project ""
+			(project "treble"
 				(path "/3f5034ce-32a3-409e-b32c-964723436806"
 					(reference "#FLG01")
@@
 		)
 		(instances
-			(project ""
+			(project "treble"
 				(path "/3f5034ce-32a3-409e-b32c-964723436806"
 					(reference "#FLG02")
@@
 		)
 		(instances
-			(project ""
+			(project "treble"
 				(path "/3f5034ce-32a3-409e-b32c-964723436806"
 					(reference "#PWR05")
@@
 		)
 		(instances
-			(project ""
+			(project "treble"
 				(path "/3f5034ce-32a3-409e-b32c-964723436806"
 					(reference "#PWR02")
@@
 		)
 		(instances
-			(project ""
+			(project "treble"
 				(path "/3f5034ce-32a3-409e-b32c-964723436806"
 					(reference "#PWR010")
@@
 		)
 		(instances
-			(project ""
+			(project "treble"
 				(path "/3f5034ce-32a3-409e-b32c-964723436806"
 					(reference "#PWR07")
@@
 		)
 		(instances
-			(project ""
+			(project "treble"
 				(path "/3f5034ce-32a3-409e-b32c-964723436806"
 					(reference "J4")
@@
 		)
 		(instances
-			(project ""
+			(project "treble"
 				(path "/3f5034ce-32a3-409e-b32c-964723436806"
 					(reference "J3")
@@
 		)
 		(instances
-			(project ""
+			(project "treble"
 				(path "/3f5034ce-32a3-409e-b32c-964723436806"
 					(reference "#PWR06")
